File: PCB/Test-PCB.kicad_sch (KiCad schematic)
At the start: 37 parts, among them J1 CNP701 (front panel), J2 CN701 (MainBoard), J3 CNP702 (front panel), J4 CN702 (MainBoard), J5 SPDIF, U1 ESP32-S3-MINI-1, U2 ESP32-S3-MINI-1, U3 SN74LVC245APW

Commit message: Add files via upload
Parts:
- added AST, BLN, CE, CLK, D-IN, DATA, MUTE, RDS-C, RDS-D, SI, ST: TestPoint, symbol Connector:TestPoint
Connections:
- net at J1.9 (Pin_9), JP1.1 (A): now also CE.1
- net at J3.4 (Pin_4), JP9.3 (B): now also AST.1
- net at J3.6 (Pin_6), JP8.3 (B): now also RDS-D.1
- net at J1.5 (Pin_5), JP5.1 (A): now also RDS-C.1
- net at J1.6 (Pin_6), JP4.1 (A): now also CLK.1
- net at J1.7 (Pin_7), JP3.1 (A): now also DATA.1
- net at J1.8 (Pin_8), JP2.1 (A): now also D-IN.1
- net at J3.1 (Pin_1), JP6.3 (B): now also BLN.1
- net at J3.7 (Pin_7), JP11.3 (B): now also SI.1
- net at J3.2 (Pin_2), JP7.3 (B): now also ST.1
- net at J3.5 (Pin_5), JP10.3 (B): now also MUTE.1

Commit message: Add files via upload
Parts:
- removed C1: 100nF, symbol Device:C
- added C2: 10uF, symbol Device:C
- added C3: 22uF, symbol Device:C
- added C4, C5, C6: 100nF, symbol Device:C
- added JP13, JP14: 3.3v ESP Enable switch, symbol Jumper:Jumper_2_Open
- added unit 5 of U3
- added unit 5 of U4
- U3: renamed from RDS-C; value 74AHCT125 -> SN74AHCT125PW
- U3: renamed from D-IN; value 74AHCT125 -> SN74AHCT125PW
- U4: renamed from RDS-D; value 74AHCT125 -> SN74AHCT125PW
- U4: renamed from ST; value 74AHCT125 -> SN74AHCT125PW
- U4: renamed from AST; value 74AHCT125 -> SN74AHCT125PW
- U4: renamed from SI; value 74AHCT125 -> SN74AHCT125PW
Connections:
- net GND: now also J5.2 (Pin_2), U3.19 (~{OE}), U3.4, U4.10, U4.13, U4.4, C2.2, C3.2, C4.2, C5.1, C6.1, U3.7 (GND), U4.2 (GND), U4.7 (GND); no longer J5.1 (Pin_1), U3.1, U4.1, U4.1, U4.1
- net SIG: now reaches U2.22 (IO18)
- net SIG: now also J5.3 (Pin_3); no longer J5.2 (Pin_2)
- net at U2.3 (3V3): now also JP13.2 (B)
- net at R4.1: now also U4.6; no longer U4.3
- net RDS-D: now reaches U1.15 (IO11)
- net RDS-D: now also U4.5; no longer U4.2
- net SI: now reaches U1.13 (IO9), U4.2
- net RDS-C: now reaches U1.16 (IO12)
- net RDS-C: now also U3.5; no longer U3.2
- net D-IN: now reaches U1.22 (IO18), U3.2
- net at U1.3 (3V3): now also JP14.2 (B)
- net ST: now reaches U1.44 (IO46)
- net ST: now also U4.12; no longer U4.2
- net AST: now reaches U1.7 (IO3)
- net AST: now also U4.9; no longer U4.2
- net at R6.2: now also U4.11; no longer U4.3
- net at R2.2: now also U3.6; no longer U3.3
- net at R5.2: now also U4.8; no longer U4.3
- net +3.3v: now reaches U3.1 (DIR)
- net +3.3v: now also U3.20 (VCC), C3.1, C4.1, JP13.1 (A), JP14.1 (A), U4.3 (VO)
- net +5V renamed +5v
- net +5v: now also J5.1 (Pin_1), C2.1, C5.2, C6.2, U3.14 (VCC), U4.1 (VI), U4.14 (VCC); no longer J5.3 (Pin_3), U3.20 (VCC)
Other:
- moved on the sheet: AST, BLN, CE, CLK, D-IN, DATA, J1, J2, J3, J4, J5, JP1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

Commit message: Add files via upload
Parts:
- J5: value SPDIF -> SPDIF-OUT
- U1: value ESP32-S3-MINI-1 -> ESP32-S3-CONTROL
- U2: value ESP32-S3-MINI-1 -> ESP32-S3-AUDIO
Connections:
- net BLN: now also U1.14 (IO10), U3.14 (B5)
- net CE: now also U1.19 (IO15), U3.18 (B1)
- net CLK: now also U1.20 (IO16), U3.16 (B3)
- net DATA: now also U1.21 (IO17), U3.17 (B2)
- net MUTE: now also U1.12 (IO8), U3.15 (B4)
- net SIG renamed OPTICAL
Changed lines of the file:
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@@
 	(wire
 		(pts
-			(xy 170.18 175.26) (xy 119.38 175.26)
-		)
-		(stroke
-			(width 0)
-			(type default)
-		)
-	)
-	(wire
-		(pts
 			(xy 201.93 132.08) (xy 210.82 132.08)
 		)
@@
 	(wire
 		(pts
-			(xy 181.61 175.26) (xy 170.18 175.26)
-		)
-		(stroke
-			(width 0)
-			(type default)
-		)
-	)
-	(wire
-		(pts
 			(xy 118.11 193.04) (xy 121.92 193.04)
 		)
@@
 	(wire
 		(pts
+			(xy 119.38 175.26) (xy 181.61 175.26)
+		)
+		(stroke
+			(width 0)
+			(type default)
+		)
+	)
+	(wire
+		(pts
 			(xy 203.2 119.38) (xy 215.9 119.38)
 		)
@@
 		)
 	)
+	(label "DATA"
+		(at 261.62 180.34 180)
+		(effects
+			(font
+				(size 1.27 1.27)
+			)
+			(justify right bottom)
+		)
+	)
+	(label "RDS-D"
+		(at 261.62 165.1 180)
+		(effects
+			(font
+				(size 1.27 1.27)
+			)
+			(justify right bottom)
+		)
+	)
 	(label "+5v"
 		(at 167.64 50.8 180)
@@
 		)
 	)
+	(label "BLN"
+		(at 261.62 162.56 180)
+		(effects
+			(font
+				(size 1.27 1.27)
+			)
+			(justify right bottom)
+		)
+	)
 	(label "+3.3v"
 		(at 182.88 50.8 0)
@@
 		)
 	)
+	(label "CE"
+		(at 261.62 175.26 180)
+		(effects
+			(font
+				(size 1.27 1.27)
+			)
+			(justify right bottom)
+		)
+	)
 	(label "RDS-D"
 		(at 213.36 204.47 180)
@@
 		)
 	)
+	(label "MUTE"
+		(at 261.62 157.48 180)
+		(effects
+			(font
+				(size 1.27 1.27)
+			)
+			(justify right bottom)
+		)
+	)
 	(label "AST"
 		(at 209.55 218.44 180)
@@
 		)
 	)
+	(label "D-IN"
+		(at 261.62 182.88 180)
+		(effects
+			(font
+				(size 1.27 1.27)
+			)
+			(justify right bottom)
+		)
+	)
+	(label "RDS-C"
+		(at 261.62 167.64 180)
+		(effects
+			(font
+				(size 1.27 1.27)
+			)
+			(justify right bottom)
+		)
+	)
 	(label "5v"
 		(at 185.42 78.74 180)
@@
 		)
 	)
+	(label "AST"
+		(at 261.62 144.78 180)
+		(effects
+			(font
+				(size 1.27 1.27)
+			)
+			(justify right bottom)
+		)
+	)
 	(label "CE"
 		(at 176.53 137.16 180)
@@
 		)
 	)
+	(label "SI/SIG"
+		(at 261.62 160.02 180)
+		(effects
+			(font
+				(size 1.27 1.27)
+			)
+			(justify right bottom)
+		)
+	)
 	(label "D-IN"
 		(at 209.55 92.71 180)
@@
 		)
 	)
+	(label "ST"
+		(at 292.1 177.8 0)
+		(effects
+			(font
+				(size 1.27 1.27)
+			)
+			(justify left bottom)
+		)
+	)
 	(label "DATA"
 		(at 176.53 139.7 180)
@@
 		)
 	)
+	(label "OPTICAL"
+		(at 261.62 115.57 180)
+		(effects
+			(font
+				(size 1.27 1.27)
+			)
+			(justify right bottom)
+		)
+	)
 	(label "5v"
-		(at 162.56 175.26 0)
+		(at 179.07 175.26 0)
 		(effects
 			(font
@@
 		)
 	)
+	(label "CLK"
+		(at 261.62 177.8 180)
+		(effects
+			(font
+				(size 1.27 1.27)
+			)
+			(justify right bottom)
+		)
+	)
 	(symbol
 		(lib_id "Jumper:Jumper_3_Bridged12")
@@
 		(in_pos_files yes)
 		(dnp no)
-		(fields_autoplaced yes)
 		(property "Reference" "C5"
-			(at 173.99 170.1799 0)
+			(at 164.846 172.974 0)
 			(show_name no)
 			(do_not_autoplace no)
@@
 		)
 		(property "Value" "100nF"
-			(at 173.99 172.7199 0)
+			(at 161.798 170.18 0)
 			(show_name no)
 			(do_not_autoplace no)
@@
 			)
 		)
-		(property "Value" "ESP32-S3-MINI-1"
+		(property "Value" "ESP32-S3-AUDIO"
 			(at 279.0033 59.69 0)
 			(show_name no)
@@
 		(in_pos_files yes)
 		(dnp no)
-		(fields_autoplaced yes)
 		(property "Reference" "R4"
-			(at 172.72 198.12 90)
+			(at 172.72 201.93 90)
 			(show_name no)
 			(do_not_autoplace no)
@@
 		)
 		(property "Value" "470Ω"
-			(at 172.72 200.66 90)
+			(at 172.72 207.01 90)
 			(show_name no)
 			(do_not_autoplace no)
@@
 			)
 		)
-		(property "Value" "ESP32-S3-MINI-1"
+		(property "Value" "ESP32-S3-CONTROL"
 			(at 279.0033 127 0)
 			(show_name no)
@@
 		(in_pos_files yes)
 		(dnp no)
-		(fields_autoplaced yes)
 		(property "Reference" "R3"
-			(at 172.72 182.88 90)
+			(at 172.72 186.944 90)
 			(show_name no)
 			(do_not_autoplace no)
@@
 		)
 		(property "Value" "470Ω"
-			(at 172.72 185.42 90)
+			(at 172.466 191.77 90)
 			(show_name no)
 			(do_not_autoplace no)
@@
 		(fields_autoplaced yes)
 		(property "Reference" "J5"
-			(at 252.095 41.9099 90)
+			(at 251.46 41.9099 90)
 			(show_name no)
 			(do_not_autoplace no)
@@
 			)
 		)
-		(property "Value" "SPDIF"
-			(at 252.095 44.4499 90)
+		(property "Value" "SPDIF-OUT"
+			(at 251.46 44.4499 90)
 			(show_name no)
 			(do_not_autoplace no)
@@
 		(in_pos_files yes)
 		(dnp no)
-		(fields_autoplaced yes)
 		(property "Reference" "R6"
-			(at 172.72 226.06 90)
+			(at 172.466 229.87 90)
 			(show_name no)
 			(do_not_autoplace no)
@@
 		)
 		(property "Value" "470Ω"
-			(at 172.72 228.6 90)
+			(at 172.974 234.95 90)
 			(show_name no)
 			(do_not_autoplace no)

Commit message: Add files via upload
Parts:
- added R12: 10k, symbol Device:R
Connections:
- net GND: now also R12.1
- net AUDIO_RESET: now reaches U2.20 (IO16)
- net AUDIO_RESET: now also U1.18 (IO14)
- net AUDIO_READY: now reaches U2.21 (IO17)
- net AUDIO_READY: now also U1.17 (IO13), R12.2
Changed lines of the file:
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@@
 	)
 	(junction
+		(at 245.11 134.62)
+		(diameter 0)
+		(color 0 0 0 0)
+	)
+	(junction
 		(at 90.17 203.2)
 		(diameter 0)
@@
 	)
 	(junction
+		(at 210.82 134.62)
+		(diameter 0)
+		(color 0 0 0 0)
+	)
+	(junction
 		(at 121.92 193.04)
 		(diameter 0)
@@
 	(wire
 		(pts
+			(xy 210.82 134.62) (xy 210.82 162.56)
+		)
+		(stroke
+			(width 0.3048)
+			(type default)
+		)
+	)
+	(wire
+		(pts
 			(xy 167.64 50.8) (xy 158.75 50.8)
 		)
@@
 	(wire
 		(pts
+			(xy 261.62 170.18) (xy 245.11 170.18)
+		)
+		(stroke
+			(width 0)
+			(type default)
+		)
+	)
+	(wire
+		(pts
 			(xy 82.55 92.71) (xy 173.99 92.71)
 		)
@@
 	(wire
 		(pts
+			(xy 238.76 134.62) (xy 245.11 134.62)
+		)
+		(stroke
+			(width 0)
+			(type default)
+		)
+	)
+	(wire
+		(pts
 			(xy 63.5 143.51) (xy 97.79 143.51)
 		)
@@
 		)
 		(stroke
-			(width 0)
+			(width 0.3048)
 			(type default)
 		)
@@
 	(wire
 		(pts
+			(xy 245.11 134.62) (xy 245.11 170.18)
+		)
+		(stroke
+			(width 0)
+			(type default)
+		)
+	)
+	(wire
+		(pts
 			(xy 175.26 58.42) (xy 190.5 58.42)
 		)
@@
 	(wire
 		(pts
-			(xy 151.13 144.78) (xy 160.02 144.78)
+			(xy 245.11 113.03) (xy 261.62 113.03)
 		)
 		(stroke
@@
 	(wire
 		(pts
-			(xy 205.74 204.47) (xy 229.87 204.47)
+			(xy 151.13 144.78) (xy 160.02 144.78)
 		)
 		(stroke
@@
 	(wire
 		(pts
-			(xy 156.21 90.17) (xy 156.21 137.16)
+			(xy 205.74 204.47) (xy 229.87 204.47)
 		)
 		(stroke
@@
 	(wire
 		(pts
-			(xy 110.49 195.58) (xy 130.81 195.58)
+			(xy 156.21 90.17) (xy 156.21 137.16)
 		)
 		(stroke
@@
 	(wire
 		(pts
-			(xy 226.06 58.42) (xy 215.9 58.42)
+			(xy 110.49 195.58) (xy 130.81 195.58)
 		)
 		(stroke
@@
 	(wire
 		(pts
-			(xy 215.9 68.58) (xy 226.06 68.58)
+			(xy 226.06 58.42) (xy 215.9 58.42)
 		)
 		(stroke
@@
 	(wire
 		(pts
-			(xy 210.82 127) (xy 210.82 132.08)
+			(xy 215.9 68.58) (xy 226.06 68.58)
 		)
 		(stroke
-			(width 0.3048)
+			(width 0)
 			(type default)
 		)
@@
 	(wire
 		(pts
-			(xy 210.82 132.08) (xy 210.82 162.56)
+			(xy 210.82 132.08) (xy 210.82 134.62)
 		)
 		(stroke
@@
 	(wire
 		(pts
+			(xy 261.62 172.72) (xy 242.57 172.72)
+		)
+		(stroke
+			(width 0)
+			(type default)
+		)
+	)
+	(wire
+		(pts
 			(xy 102.87 97.79) (xy 151.13 97.79)
 		)
@@
 	(wire
 		(pts
+			(xy 242.57 110.49) (xy 261.62 110.49)
+		)
+		(stroke
+			(width 0)
+			(type default)
+		)
+	)
+	(wire
+		(pts
 			(xy 203.2 119.38) (xy 215.9 119.38)
 		)
@@
 	(wire
 		(pts
+			(xy 210.82 127) (xy 210.82 132.08)
+		)
+		(stroke
+			(width 0.3048)
+			(type default)
+		)
+	)
+	(wire
+		(pts
 			(xy 151.13 220.98) (xy 151.13 144.78)
 		)
@@
 		)
 		(stroke
-			(width 0)
+			(width 0.3048)
 			(type default)
 		)
@@
 	(wire
 		(pts
+			(xy 210.82 134.62) (xy 231.14 134.62)
+		)
+		(stroke
+			(width 0)
+			(type default)
+		)
+	)
+	(wire
+		(pts
 			(xy 63.5 190.5) (xy 119.38 190.5)
 		)
@@
 	(wire
 		(pts
+			(xy 245.11 113.03) (xy 245.11 134.62)
+		)
+		(stroke
+			(width 0)
+			(type default)
+		)
+	)
+	(wire
+		(pts
 			(xy 72.39 209.55) (xy 72.39 228.6)
 		)
@@
 	(wire
 		(pts
+			(xy 242.57 110.49) (xy 242.57 172.72)
+		)
+		(stroke
+			(width 0)
+			(type default)
+		)
+	)
+	(wire
+		(pts
 			(xy 63.5 205.74) (xy 67.31 205.74)
 		)
@@
 		)
 	)
+	(label "AUDIO_RESET"
+		(at 261.62 110.49 180)
+		(effects
+			(font
+				(size 1.27 1.27)
+			)
+			(justify right bottom)
+		)
+	)
 	(label "AST"
 		(at 209.55 218.44 180)
@@
 		)
 	)
+	(label "AUDIO_READY"
+		(at 261.62 113.03 180)
+		(effects
+			(font
+				(size 1.27 1.27)
+			)
+			(justify right bottom)
+		)
+	)
 	(label "RDS-C"
 		(at 212.09 110.49 180)
@@
 	)
 	(symbol
+		(lib_id "Device:R")
+		(at 234.95 134.62 90)
+		(unit 1)
+		(body_style 1)
+		(exclude_from_sim no)
+		(in_bom yes)
+		(on_board yes)
+		(in_pos_files yes)
+		(dnp no)
+		(property "Reference" "R12"
+			(at 234.95 136.906 90)
+			(show_name no)
+			(do_not_autoplace no)
+			(effects
+				(font
+					(size 1.27 1.27)
+				)
+			)
+		)
+		(property "Value" "10k"
+			(at 234.95 134.62 90)
+			(show_name no)
+			(do_not_autoplace no)
+			(effects
+				(font
+					(size 1.27 1.27)
+				)
+			)
+		)
+		(property "Footprint" ""
+			(at 234.95 136.398 90)
+			(hide yes)
+			(show_name no)
+			(do_not_autoplace no)
+			(effects
+				(font
+					(size 1.27 1.27)
+				)
+			)
+		)
+		(property "Datasheet" ""
+			(at 234.95 134.62 0)
+			(hide yes)
+			(show_name no)
+			(do_not_autoplace no)
+			(effects
+				(font
+					(size 1.27 1.27)
+				)
+			)
+		)
+		(property "Description" "Resistor"
+			(at 234.95 134.62 0)
+			(hide yes)
+			(show_name no)
+			(do_not_autoplace no)
+			(effects
+				(font
+					(size 1.27 1.27)
+				)
+			)
+		)
+		(pin "2"
+		)
+		(pin "1"
+		)
+		(instances
+			(project "Test-PCB"
+				(path "/5d6697d5-c0bf-4044-ac4e-730c1ec0afe4"
+					(reference "R12")
+					(unit 1)
+				)
+			)
+		)
+	)
+	(symbol
 		(lib_id "Jumper:Jumper_2_Open")
 		(at 231.14 68.58 0)
@@
 		(dnp no)
 		(property "Reference" "U4"
-			(at 195.834 198.12 0)
+			(at 199.644 204.47 0)
 			(show_name no)
 			(do_not_autoplace no)
@@
 		(property "Value" "SN74AHCT125PW"
 			(at 193.548 200.406 0)
+			(hide yes)
 			(show_name no)
 			(do_not_autoplace no)
@@
 		(dnp no)
 		(property "Reference" "U4"
-			(at 195.58 226.06 0)
+			(at 199.39 232.41 0)
 			(show_name no)
 			(do_not_autoplace no)
@@
 		)
 		(property "Value" "SN74AHCT125PW"
-			(at 192.024 228.6 0)
+			(at 194.818 182.88 0)
 			(show_name no)
 			(do_not_autoplace no)
@@
 		(dnp no)
 		(property "Reference" "U3"
-			(at 185.674 109.22 0)
+			(at 197.866 110.49 0)
 			(show_name no)
 			(do_not_autoplace no)
@@
 		(property "Value" "SN74AHCT125PW"
 			(at 179.832 111.506 0)
+			(hide yes)
 			(show_name no)
 			(do_not_autoplace no)
@@
 		(dnp no)
 		(property "Reference" "U3"
-			(at 195.326 69.088 90)
+			(at 190.754 65.278 90)
 			(show_name no)
 			(do_not_autoplace no)
@@
 		)
 		(property "Value" "SN74AHCT125PW"
-			(at 198.628 71.882 90)
+			(at 199.136 69.596 90)
 			(show_name no)
 			(do_not_autoplace no)
@@
 		(dnp no)
 		(property "Reference" "U4"
-			(at 183.388 171.958 90)
+			(at 194.31 166.37 90)
 			(show_name no)
 			(do_not_autoplace no)
@@
 		(property "Value" "SN74AHCT125PW"
 			(at 178.308 177.292 90)
+			(hide yes)
 			(show_name no)
 			(do_not_autoplace no)
@@
 		(dnp no)
 		(property "Reference" "U4"
-			(at 194.31 212.344 0)
+			(at 199.644 218.186 0)
 			(show_name no)
 			(do_not_autoplace no)
@@
 		(property "Value" "SN74AHCT125PW"
 			(at 193.294 214.376 0)
+			(hide yes)
 			(show_name no)
 			(do_not_autoplace no)
@@
 		(dnp no)
 		(property "Reference" "U4"
-			(at 196.342 183.642 0)
+			(at 199.39 189.23 0)
 			(show_name no)
 			(do_not_autoplace no)
@@
 		(property "Value" "SN74AHCT125PW"
 			(at 191.516 185.928 0)
+			(hide yes)
 			(show_name no)
 			(do_not_autoplace no)
@@
 		(dnp no)
 		(property "Reference" "U3"
-			(at 196.85 86.106 0)
+			(at 198.374 92.456 0)
 			(show_name no)
 			(do_not_autoplace no)
@@
 		(property "Value" "SN74AHCT125PW"
 			(at 191.008 88.392 0)
+			(hide yes)
 			(show_name no)
 			(do_not_autoplace no)

Commit message: Add files via upload
Parts:
- removed AST, BLN, CE, CLK, D-IN, DATA, MUTE, RDS-C, RDS-D, SI, ST: TestPoint, symbol Connector:TestPoint
- renumbered U4 to U5
Connections:
- net AST: now also J3.4 (Pin_4), JP9.2 (C)
- net BLN: now also J3.1 (Pin_1), JP6.2 (C)
- net CE: now also J1.9 (Pin_9), JP1.2 (C)
- net CLK: now also J1.6 (Pin_6), JP4.2 (C)
- net D-IN: now also J1.8 (Pin_8), JP2.2 (C)
- net DATA: now also J1.7 (Pin_7), JP3.2 (C)
- net MUTE: now also J3.5 (Pin_5), JP10.2 (C)
- net RDS-C: now also J1.5 (Pin_5), JP5.2 (C)
- net RDS-D: now also J3.6 (Pin_6), JP8.2 (C), U1.13 (IO9), U4.2
- net SI: now also J3.7 (Pin_7); no longer U1.13 (IO9), U4.2
- net ST: now also J3.2 (Pin_2), JP7.2 (C)
- net at JP1.1 (A): now also J2.9 (Pin_9); no longer J1.9 (Pin_9)
- net at R7.1: now also JP1.3 (B); no longer JP1.2 (C)
- net at JP9.1 (A): now also R5.1; no longer J4.4 (Pin_4)
- net at JP9.3 (B): now also J4.4 (Pin_4); no longer J3.4 (Pin_4)
- net at JP8.1 (A): now also R4.2; no longer J4.6 (Pin_6)
- net at JP8.3 (B): now also J4.6 (Pin_6); no longer J3.6 (Pin_6)
- net at JP4.1 (A): now also J2.6 (Pin_6); no longer J1.6 (Pin_6)
- net 30V: now reaches J1.1 (Pin_1), J2.1 (Pin_1)
- net POWER: now reaches J1.4 (Pin_4), J2.4 (Pin_4)
- net at JP5.1 (A): now also J2.5 (Pin_5); no longer J1.5 (Pin_5)
- net at JP3.1 (A): now also J2.7 (Pin_7); no longer J1.7 (Pin_7)
- net at JP2.1 (A): now also J2.8 (Pin_8); no longer J1.8 (Pin_8)
- net at JP6.1 (A): now also R11.1; no longer J4.1 (Pin_1)
- net at JP6.3 (B): now also J4.1 (Pin_1); no longer J3.1 (Pin_1)
- net at JP7.3 (B): now also J4.2 (Pin_2); no longer J3.2 (Pin_2)
- net at JP5.3 (B): now also R2.1; no longer J2.5 (Pin_5)
- net at JP4.3 (B): now also R9.1; no longer J2.6 (Pin_6)
- net at JP3.3 (B): now also R8.1; no longer J2.7 (Pin_7)
- net at JP2.3 (B): now also R1.1; no longer J2.8 (Pin_8)
- net at JP11.1 (A): now also R3.1; no longer J4.7 (Pin_7)
- net at JP11.2 (C): no longer R3.1
- net at JP11.3 (B): now also J4.7 (Pin_7); no longer J3.7 (Pin_7)
- net at R10.1: now also JP10.1 (A); no longer JP10.2 (C)
- net at JP10.3 (B): now also J4.5 (Pin_5); no longer J3.5 (Pin_5)
- net at JP7.1 (A): now also R6.1; no longer J4.2 (Pin_2)
- net n/a: now reaches J3.3 (Pin_3)
- net FL: now reaches J3.8 (Pin_8), J4.8 (Pin_8)
- net FL: now also J3.9 (Pin_9), J4.9 (Pin_9)
- net +5v renamed +5V
Other:
- moved on the sheet: J1, J4, JP1, JP10, JP11, JP2, JP3, JP4, JP5, JP6, JP7, JP8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

Commit message: Add files via upload
Connections:
- net GND is gone; now on net +5V: C2.2, C3.2, C4.2, C5.1, C6.1, J1.3 (Pin_3), J2.3 (Pin_3), J5.2 (Pin_2), R12.1, U1.1 (GND), U1.2 (GND), U1.42 (GND), U1.43 (GND), U1.46 (GND), U1.47 (GND), U1.48 (GND), U1.49 (GND), U1.50 (GND), U1.51 (GND), U1.52 (GND), U1.53 (GND), U1.54 (GND), U1.55 (GND), U1.56 (GND), U1.57 (GND), U1.58 (GND), U1.59 (GND), U1.60 (GND), U1.61 (GND), U1.62 (GND), U1.63 (GND), U1.64 (GND), U1.65 (GND), U2.1 (GND), U2.2 (GND), U2.42 (GND), U2.43 (GND), U2.46 (GND), U2.47 (GND), U2.48 (GND), U2.49 (GND), U2.50 (GND), U2.51 (GND), U2.52 (GND), U2.53 (GND), U2.54 (GND), U2.55 (GND), U2.56 (GND), U2.57 (GND), U2.58 (GND), U2.59 (GND), U2.60 (GND), U2.61 (GND), U2.62 (GND), U2.63 (GND), U2.64 (GND), U2.65 (GND), U3.1, U3.10 (GND), U3.19 (~{OE}), U3.4, U3.7 (GND), U4.1, U4.10, U4.13, U4.4, U4.7 (GND), U5.2 (GND)
Changed lines of the file:
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@@
+	)
+	(junction
+		(at 119.38 151.13)
+		(diameter 0)
+		(color 0 0 0 0)
 	)
 	(junction
@@
 	(wire
 		(pts
+			(xy 119.38 151.13) (xy 119.38 175.26)
+		)
+		(stroke
+			(width 0)
+			(type default)
+		)
+	)
+	(wire
+		(pts
 			(xy 153.67 95.25) (xy 153.67 139.7)
 		)
@@
 	(wire
 		(pts
-			(xy 63.5 151.13) (xy 134.62 151.13)
+			(xy 63.5 151.13) (xy 119.38 151.13)
 		)
 		(stroke
@@
 		(stroke
 			(width 0)
+			(type default)
+		)
+	)
+	(wire
+		(pts
+			(xy 119.38 151.13) (xy 134.62 151.13)
+		)
+		(stroke
+			(width 0.3048)
 			(type default)
 		)
@@
 		(dnp no)
 		(property "Reference" "J1"
-			(at 150.622 137.16 0)
-			(show_name no)
-			(do_not_autoplace no)
+			(at 147.32 133.35 0)
+			(show_name no)
+			(do_not_autoplace no)

Commit message: Add files via upload
Connections:
- net RDS-D: no longer U1.13 (IO9), U4.2
- net SI: now also U1.13 (IO9), U4.2
Changed lines of the file:
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@@
+	(wire
+		(pts
+			(xy 205.74 189.23) (xy 227.33 189.23)
+		)
+		(stroke
+			(width 0)
+			(type default)
+		)
+	)
 	(wire
 		(pts
@@
 		(pts
 			(xy 168.91 119.38) (xy 189.23 119.38)
-		)
-		(stroke
-			(width 0)
-			(type default)
-		)
-	)
-	(wire
-		(pts
-			(xy 205.74 189.23) (xy 227.33 189.23)
 		)
 		(stroke
@@
 		)
 	)
-	(label "RDS-D"
-		(at 213.36 189.23 180)
-		(effects
-			(font
-				(size 1.27 1.27)
-			)
-			(justify right bottom)
-		)
-	)
 	(label "FL"
 		(at 130.81 185.42 180)
@@
 	)
 	(label "RDS-D"
-		(at 208.28 204.47 180)
+		(at 213.36 204.47 180)
 		(effects
 			(font
@@
 	(label "ST"
 		(at 130.81 203.2 180)
+		(effects
+			(font
+				(size 1.27 1.27)
+			)
+			(justify right bottom)
+		)
+	)
+	(label "SI"
+		(at 208.28 189.23 180)
 		(effects
 			(font
@@
 		(dnp no)
 		(property "Reference" "J1"
-			(at 147.32 133.35 0)
-			(show_name no)
-			(do_not_autoplace no)
+			(at 150.622 137.16 0)
+			(show_name no)
+			(do_not_autoplace no)

Commit message: Add files via upload
Connections:
- net +5V: no longer C2.2, C3.2, C4.2, C5.1, C6.1, J1.3 (Pin_3), J2.3 (Pin_3), J5.2 (Pin_2), R12.1, U1.1 (GND), U1.2 (GND), U1.42 (GND), U1.43 (GND), U1.46 (GND), U1.47 (GND), U1.48 (GND), U1.49 (GND), U1.50 (GND), U1.51 (GND), U1.52 (GND), U1.53 (GND), U1.54 (GND), U1.55 (GND), U1.56 (GND), U1.57 (GND), U1.58 (GND), U1.59 (GND), U1.60 (GND), U1.61 (GND), U1.62 (GND), U1.63 (GND), U1.64 (GND), U1.65 (GND), U2.1 (GND), U2.2 (GND), U2.42 (GND), U2.43 (GND), U2.46 (GND), U2.47 (GND), U2.48 (GND), U2.49 (GND), U2.50 (GND), U2.51 (GND), U2.52 (GND), U2.53 (GND), U2.54 (GND), U2.55 (GND), U2.56 (GND), U2.57 (GND), U2.58 (GND), U2.59 (GND), U2.60 (GND), U2.61 (GND), U2.62 (GND), U2.63 (GND), U2.64 (GND), U2.65 (GND), U3.1, U3.10 (GND), U3.19 (~{OE}), U3.4, U3.7 (GND), U4.1, U4.10, U4.13, U4.4, U4.7 (GND), U5.2 (GND)
- new net GND: C2.2, C3.2, C4.2, C5.1, C6.1, J1.3 (Pin_3), J2.3 (Pin_3), J5.2 (Pin_2), R12.1, U1.1 (GND), U1.2 (GND), U1.42 (GND), U1.43 (GND), U1.46 (GND), U1.47 (GND), U1.48 (GND), U1.49 (GND), U1.50 (GND), U1.51 (GND), U1.52 (GND), U1.53 (GND), U1.54 (GND), U1.55 (GND), U1.56 (GND), U1.57 (GND), U1.58 (GND), U1.59 (GND), U1.60 (GND), U1.61 (GND), U1.62 (GND), U1.63 (GND), U1.64 (GND), U1.65 (GND), U2.1 (GND), U2.2 (GND), U2.42 (GND), U2.43 (GND), U2.46 (GND), U2.47 (GND), U2.48 (GND), U2.49 (GND), U2.50 (GND), U2.51 (GND), U2.52 (GND), U2.53 (GND), U2.54 (GND), U2.55 (GND), U2.56 (GND), U2.57 (GND), U2.58 (GND), U2.59 (GND), U2.60 (GND), U2.61 (GND), U2.62 (GND), U2.63 (GND), U2.64 (GND), U2.65 (GND), U3.1, U3.10 (GND), U3.19 (~{OE}), U3.4, U3.7 (GND), U4.1, U4.10, U4.13, U4.4, U4.7 (GND), U5.2 (GND)
